Commit message: make ros node work with any number of actuators and states

File: src/pupper_rviz/urdf/pupper_v3.urdf (robot description, URDF)
Before this commit: robot pupper_v3, 13 links, 12 joints
Links:
- link base_link: geometry collision box size=0.24018 0.10194 0.115; visual mesh filename=package://pupper_rviz/meshes/dae/ProtoAssembly-MGv25.004.dae scale=1.0 1.0 1.0
- link leg_back_l_1: geometry visual mesh filename=package://pupper_rviz/meshes/dae/ProtoAssembly-MGv25.016.dae scale=1.0 1.0 1.0
- link leg_back_l_2: geometry visual mesh filename=package://pupper_rviz/meshes/dae/ProtoAssembly-MGv25.014.dae scale=1.0 1.0 1.0
- link leg_back_l_3: geometry collision sphere radius=0.01984; visual mesh filename=package://pupper_rviz/meshes/dae/ProtoAssembly-MGv25.015.dae scale=1.0 1.0 1.0
- link leg_back_r_1: geometry visual mesh filename=package://pupper_rviz/meshes/dae/ProtoAssembly-MGv25.012.dae scale=1.0 1.0 1.0
- link leg_back_r_2: geometry visual mesh filename=package://pupper_rviz/meshes/dae/ProtoAssembly-MGv25.010.dae scale=1.0 1.0 1.0
- link leg_back_r_3: geometry collision sphere radius=0.01984; visual mesh filename=package://pupper_rviz/meshes/dae/ProtoAssembly-MGv25.011.dae scale=1.0 1.0 1.0
- link leg_front_l_1: geometry visual mesh filename=package://pupper_rviz/meshes/dae/ProtoAssembly-MGv25.003.dae scale=1.0 1.0 1.0
- link leg_front_l_2: geometry visual mesh filename=package://pupper_rviz/meshes/dae/ProtoAssembly-MGv25.001.dae scale=1.0 1.0 1.0
- link leg_front_l_3: geometry collision sphere radius=0.01984; visual mesh filename=package://pupper_rviz/meshes/dae/ProtoAssembly-MGv25.002.dae scale=1.0 1.0 1.0
- link leg_front_r_1: geometry visual mesh filename=package://pupper_rviz/meshes/dae/ProtoAssembly-MGv25.007.dae scale=1.0 1.0 1.0
- link leg_front_r_2: geometry visual mesh filename=package://pupper_rviz/meshes/dae/ProtoAssembly-MGv25.005.dae scale=1.0 1.0 1.0
- link leg_front_r_3: geometry collision sphere radius=0.01984; visual mesh filename=package://pupper_rviz/meshes/dae/ProtoAssembly-MGv25.006.dae scale=1.0 1.0 1.0
